File: hardware/external-antenna/cad/mc2.kicad_pcb (KiCad board)
At the start: 2 copper layers, 100 x 100 mm, 25 parts, among them J1 FUSED ISOLATED 5V INPUT, J2 D24V22F3 external assembled b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, J3 DFR0627 WK2132 ready module h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, J4 ZAC93 ready module harness, J5 CC1101 ready module harness, J6 LD2450 radar harness, J7 BME680 external pod harness, J8 XIAO BOOT unpopulated service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, J9 HOST BOOT unpopulated service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, U1 ESP32-DevKitC-VIE, U2 Unexpected Maker TinyC6[D] TC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, U3 Seeed XIAO MG24 pre-soldered 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, U4 WIZ850io finished module

Commit message: Migrate MC2-D to factory-header XIAO ESP32C6
Parts:
- removed R3: 10k C6 download strap GPIO8, MC2:R_Axial_DIN0207_L6.3mm_D2.5mm_P7.62mm_Horizontal
- added J10: C6 EN/BOOT underside recovery harness, MC2:PinHeader_1x02_P2.54mm_Vertical, F.Cu at (49.5, 39.0)
- J2: value D24V22F3 external assembled buck -> RECOM R-78K3.3-1.0 offboard 3V3 converter
- U2: value Unexpected Maker TinyC6[D] TC6D-01 -> Seeed XIAO ESP32C6 pre-soldered 102010636; footprint MC2:TinyC6_D -> MC2:XIAO_ESP32C6
- moved U2 16.9 mm to (46.2, 14.9)
Connections:
- U2 pad 10: /C6_STRAP8 -> unconnected-(U2-GPIO20-Pad10)
- U2 pad 11: /THREAD_BOOT -> unconnected-(U2-GPIO18-Pad11)
- U2 pad 12: /THREAD_RX -> unconnected-(U2-3V3-Pad12)
- U2 pad 13: /THREAD_TX -> /GND
- U2 pad 14: /GND -> /+5V_C6
- U2 pad 2: /GND -> unconnected-(U2-GPIO1-Pad2)
- U2 pad 3: /+5V_C6 -> unconnected-(U2-GPIO2-Pad3)
- U2 pad 4: /C6_LOCAL_3V3 -> unconnected-(U2-GPIO21-Pad4)
- U2 pad 7: unconnected-(U2-GPIO1-Pad7) -> /THREAD_TX
- U2 pad 8: unconnected-(U2-GPIO0-Pad8) -> /THREAD_RX
Routing:
- net /THREAD_RX: track 43.3 -> 65.6 mm
- net /C6_STRAP8: track 20.4 -> 0.00 mm
- net /RF_GDO2: track 57.7 -> 78.1 mm, vias 1 -> 0
- net /ETH_RESET: track 64.5 -> 47.6 mm, vias 0 -> 1
- net /ETH_CS: track 82.4 -> 65.9 mm
- net /ZB_RX: track 100.2 -> 84.3 mm
- net /THREAD_TX: track 55.8 -> 40.7 mm, vias 0 -> 1
- net /C6_LOCAL_3V3: track 12.8 -> 0.00 mm
- net /I2C_SDA: track 112.1 -> 101.6 mm, vias 0 -> 1
- net /HOST_BOOT_SERVICE: track 90.5 -> 99.5 mm, vias 0 -> 1
- net /SPI_SCK: track 107.2 -> 116.0 mm, vias 2 -> 0
- net /ZB_TX: track 76.2 -> 68.1 mm
- net /RADAR_RX: track 47.4 -> 54.0 mm
- net /RF_CS: track 94.5 -> 88.7 mm
- net /+5V_C6: track 50.8 -> 55.8 mm
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Other:
- outline, holes or cut-outs redrawn
- board text added: "MC2-D ESP32"
- board text removed: "MC2-C ESP32"

Commit message: Qualify MC2-D purchase fit and remove host feed voltage drop
Parts:
- D1: value 1N5819 USB supply isolation -> 22AWG WIRE LINK - NO DIODE; footprint MC2:D_DO-41_SOD81_P7.62mm_Horizontal -> MC2:Wire_Link_P7.62mm
