File: hardware/external-antenna/cad/mc2.kicad_pcb (KiCad board)
At the start: 2 copper layers, 100 x 100 mm, 23 parts, among them J1 FUSED ISOLATED 5V INPUT, J2 D24V22F3 external assembled b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, J3 DFR0627 WK2132 ready module h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, J4 ZAC93 ready module harness, J5 CC1101 ready module harness, J6 LD2450 radar harness, J7 BME680 external pod harness, J8 XIAO BOOT unpopulated service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, J9 S3 BOOT unpopulated service p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, U1 ESP32-S3-DevKitC-1U-N8R8, U2 Unexpected Maker TinyC6-U-01, U3 Seeed XIAO MG24 pre-soldered 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, U4 WIZ850io finished module

Commit message: Migrate MC2-B to the lower-cost classic ESP32 host (#11)
Replace the MC2-A ESP32-S3-DevKitC-1U-N8R8 host with the
previous-generation ESP32-DevKitC-VIE / WROVER-IE to reduce host
purchase cost while retaining Ethernet, local OTBR, Zigbee, three active
BLE proxy connections, Z-Wave, RF RX/TX, LD2450 and BME680. The indexed
VIE offer was $9.48 versus the previously inspected $15.20 S3 promotion,
before delivery/tax; this is not a whole-device cost or power claim.

The new **MC2-B** carrier has the exact 38-pin host footprint, a checked
21-signal map and GPIO12/GPIO2 boot pull-downs. Keep the 100×100 mm
outline and supports, so the five existing enclosure meshes remain
unchanged. Update the schematic, routed PCB, connector lookup, BOM,
assembly instructions and README appearance concepts together.

Firmware targets classic ESP32 ECOv3 at 160 MHz, quad PSRAM at 40 MHz
and node identity `mc2-classic-hub`. Check actual image target/revision,
disable the IDF console so UART0 can serve radar, and preserve UART1/2
for Zigbee/Thread. Extend the shared component guards without changing
the S3 defaults. Fix the authenticated updater's expected node name and
bind its C6 evidence to the current recipe.

Compatibility limits are explicit: **BLE 4.2**, no BLE 5 extended
advertising or Coded PHY; 8 MB physical PSRAM but at most 4 MB directly
mapped. This requires the new carrier and an initial USB-UART flash with
private configuration. S3 OTA images and MC2-A pinouts are incompatible.
No hardware was flashed or Home Assistant changed.

Validation:
- Full pinned ESPHome 2026.9.1 / ESP-IDF 5.5.5 host build:
1,708,944-byte application; 2,223,216 bytes spare in each OTA slot;
separate DRAM/IRAM evidence and image-header checks.
- 26 MC2 tests, 62 MC1 regressions, 77 shared RF/UART/migration tests,
13 MG24 recipe tests; C++ RMT lifecycle checked with ASan/UBSan.
- KiCad ERC, DRC, unconnected items and schematic parity: zero; clean
CAD reproduction passes; every pin-plan role checked agai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
Parts:
- added R4: 10k host GPIO12 SCK boot pull-down, MC2:R_Axial_DIN0207_L6.3mm_D2.5mm_P7.62mm_Horizontal, F.Cu at (8.00, 74.0)
- added R5: 10k host GPIO2 MOSI boot pull-down, MC2:R_Axial_DIN0207_L6.3mm_D2.5mm_P7.62mm_Horizontal, F.Cu at (8.00, 79.0)
- J9: value S3 BOOT unpopulated service pads -> HOST BOOT unpopulated service pads
- U1: value ESP32-S3-DevKitC-1U-N8R8 -> ESP32-DevKitC-VIE; footprint MC2:S3_DevKitC1U -> MC2:ESP32_DevKitC_VIE
- moved U1 6.60 mm to (9.27, 20.0)
Connections:
- net /S3_BOOT_SERVICE renamed /HOST_BOOT_SERVICE
- D1 pad 1: /+5V_S3 -> /+5V_HOST
- U1 pad J3.10: unconnected-(U1-GPIO38-PadJ3.10) -> /ETH_CS
- U1 pad J3.13: unconnected-(U1-GPIO35-PadJ3.13) -> /ETH_RESET
- U1 pad J3.15: unconnected-(U1-GPIO45-PadJ3.15) -> /SPI_MOSI
- U1 pad J3.16: unconnected-(U1-GPIO48-PadJ3.16) -> /THREAD_BOOT
- U1 pad J3.17: /THREAD_EN -> unconnected-(U1-GPIO8-PadJ3.17)
- U1 pad J3.18: /ZB_RTS -> unconnected-(U1-GPIO7-PadJ3.18)
- U1 pad J3.2: unconnected-(U1-GPIO43-PadJ3.2) -> /RADAR_RX
- U1 pad J3.3: unconnected-(U1-GPIO44-PadJ3.3) -> /I2C_SCL
- U1 pad J3.4: /I2C_SDA -> unconnected-(U1-GPIO1-PadJ3.4)
- U1 pad J3.5: /I2C_SCL -> unconnected-(U1-GPIO3-PadJ3.5)
- U1 pad J3.6: unconnected-(U1-GPIO42-PadJ3.6) -> /I2C_SDA
- U1 pad J3.7: unconnected-(U1-GPIO41-PadJ3.7) -> /GND
- U1 pad J3.8: /RADAR_TX -> /SPI_MISO
- U1 pad J3.9: /THREAD_BOOT -> /RADAR_TX
Routing:
- net /+5V_S3: track 43.1 -> 0.00 mm
- net /+5V_HOST: track 0.00 -> 42.4 mm
- net /RF_CS: track 122.4 -> 94.5 mm
- net /I2C_SCL: track 120.0 -> 94.2 mm, vias 0 -> 1
- net /I2C_SDA: track 91.9 -> 112.1 mm, vias 1 -> 0
- net /SPI_MISO: track 74.1 -> 54.9 mm, vias 0 -> 1
- net /GND: track 301.3 -> 320.0 mm
- net /ETH_INT: track 96.3 -> 112.3 mm, vias 1 -> 0
- net /THREAD_TX: track 40.2 -> 55.8 mm
- net /RADAR_TX: track 43.2 -> 29.1 mm
- net /RF_GDO2: track 71.4 -> 57.7 mm, vias 0 -> 1
- net /ZB_RTS: track 67.9 -> 80.8 mm, vias 1 -> 0
- net /THREAD_BOOT: track 32.6 -> 45.3 mm, vias 0 -> 1
- net /ETH_RESET: track 76.5 -> 64.5 mm
- net /RF_GDO0: track 98.8 -> 87.3 mm
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Other:
- board text added: "MC2-B ESP32"
- board text removed: "MC2 EXTERNAL"

Commit message: Match the MC2-C prototype to available TinyC6 D hardware (#17)
The original TC6-U-01 is obsolete/restricted at the checked US supplier
and has not been purchased. MC2-C selects the available TinyC6[D]
TC6D-01 and ships one matching carrier, firmware and enclosure package
for a five-board prototype order.

- Transcribe and verify the new module against pinned manufacturer
schematic, pinout and STEP files; correct its longer body, unused GPIO10
pad label, USB shell and relocated U.FL endpoint. Keep all connected
pads and copper unchanged.
- Select the external antenna through FXL6408 before Thread starts, fail
closed on configuration errors, and reject old C6 images in the updater.
Preserve the classic ESP32 host and all existing services.
- Regenerate the FH1 assembly views and print archive. All 14 printable
STL geometries remain unchanged; the corrected Thread coax route fits
the selected 150 mm cable with the specified slack.
- Publish native Gerbers, separate PTH/NPTH drill files and a manifest
that rejects stale CAD, firmware recipes, mechanical inputs and
artifacts. Add the ordering guide, current part availability and
observed quantity/shipping comparison.

Validation: native KiCad 10.0.6 ERC/DRC/unconnected/parity all zero;
clean source reproduction and unchanged-connected-copper comparison
pass. Fresh ESP32 and C6 builds pass. Firmware suites: 193 tests;
full-hub mechanics: 30 tests; fabrication/harness/guide: 24 tests.
Offline source/link/secret checks pass. Physical fit, rail headroom,
radio coexistence and coverage remain prototype commissioning work. No
purchase, device flash or Home Assistant migration has been performed.
Parts:
- U2: value Unexpected Maker TinyC6-U-01 -> Unexpected Maker TinyC6[D] TC6D-01; footprint MC2:TinyC6_U -> MC2:TinyC6_D
Other:
- board text added: "MC2-C ESP32"
- board text removed: "MC2-B ESP32"

Commit message: Use factory-header XIAO ESP32C6 and fix I2C/RF conflicts (#21)
MC2-D replaces the unpurchased TinyC6[D] with the US-distributed,
factory-header Seeed XIAO ESP32C6 (102010636), retaining the ordered
ESP32-DevKitC-VIE and the existing hub functions. The new carrier
includes the XIAO footprint, J10 recovery leads and an underside access
window; firmware and assembly models match its 4 MB flash and
external-antenna control.

An independent connection audit also found an I2C collision: the DFR0627
setting A1=1/A0=1 decodes 0x70–0x77, including BME680. Both maintained
MC2 and MC1 firmware profiles now use A1=1/A0=0, UART1 register/FIFO
0x50/0x51, reserving 0x50–0x57. Configuration validation rejects another
device in the bridge's entire address block. Assembly instructions,
current wiring graphics and CAD metadata carry the corrected switch
setting. This address correction changes no PCB copper or print
geometry.

The audit also found an RMT startup contention window on CC1101 GDO0. A
local, version-guarded initialization wrapper releases the configured RF
pin and sets HIGH idle before the driver connects its output; the shared
RF package uses it without an upstream fork or SDK cache changes. Other
transmitter pins retain their normal allocation path. Runtime handoff
also requires GDO0 high-impedance readback and confirmed IDLE/TX states
before the waveform; failed transitions release the line and skip
transmission, and RX restoration is verified.

The final purchase audit confirms all 28 submitted DigiKey lines and the
Mouser ESP32-DevKitC-VIE against the MC2-D interfaces. It also removes
the avoidable Schottky drop before the host AMS1117: the legacy D1 pads
now take an insulated 22 AWG wire link, labelled NO DIODE. D2/D3 remain
1N5819, so the third purchased diode is a spare. The copper topology is
unchanged. The assembled hub uses PoE/OTA only; host USB could feed the
full 5 V bus through the link. ZAC93 instructions explicitly require
soldering the harness to the ada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
Parts:
- removed R3: 10k C6 download strap GPIO8, MC2:R_Axial_DIN0207_L6.3mm_D2.5mm_P7.62mm_Horizontal
- added J10: C6 EN/BOOT underside recovery harness, MC2:PinHeader_1x02_P2.54mm_Vertical, F.Cu at (49.5, 39.0)
- D1: value 1N5819 USB supply isolation -> 22AWG WIRE LINK - NO DIODE; footprint MC2:D_DO-41_SOD81_P7.62mm_Horizontal -> MC2:Wire_Link_P7.62mm
- J2: value D24V22F3 external assembled buck -> RECOM R-78K3.3-1.0 offboard 3V3 converter
- U2: value Unexpected Maker TinyC6[D] TC6D-01 -> Seeed XIAO ESP32C6 pre-soldered 102010636; footprint MC2:TinyC6_D -> MC2:XIAO_ESP32C6
- moved U2 16.9 mm to (46.2, 14.9)
Connections:
- U2 pad 10: /C6_STRAP8 -> unconnected-(U2-GPIO20-Pad10)
- U2 pad 11: /THREAD_BOOT -> unconnected-(U2-GPIO18-Pad11)
- U2 pad 12: /THREAD_RX -> unconnected-(U2-3V3-Pad12)
- U2 pad 13: /THREAD_TX -> /GND
- U2 pad 14: /GND -> /+5V_C6
- U2 pad 2: /GND -> unconnected-(U2-GPIO1-Pad2)
- U2 pad 3: /+5V_C6 -> unconnected-(U2-GPIO2-Pad3)
- U2 pad 4: /C6_LOCAL_3V3 -> unconnected-(U2-GPIO21-Pad4)
- U2 pad 7: unconnected-(U2-GPIO1-Pad7) -> /THREAD_TX
- U2 pad 8: unconnected-(U2-GPIO0-Pad8) -> /THREAD_RX
Routing:
- net /THREAD_RX: track 43.3 -> 65.6 mm
- net /C6_STRAP8: track 20.4 -> 0.00 mm
- net /RF_GDO2: track 57.7 -> 78.1 mm, vias 1 -> 0
- net /ETH_RESET: track 64.5 -> 47.6 mm, vias 0 -> 1
- net /ETH_CS: track 82.4 -> 65.9 mm
- net /ZB_RX: track 100.2 -> 84.3 mm
- net /THREAD_TX: track 55.8 -> 40.7 mm, vias 0 -> 1
- net /C6_LOCAL_3V3: track 12.8 -> 0.00 mm
- net /I2C_SDA: track 112.1 -> 101.6 mm, vias 0 -> 1
- net /HOST_BOOT_SERVICE: track 90.5 -> 99.5 mm, vias 0 -> 1
- net /SPI_SCK: track 107.2 -> 116.0 mm, vias 2 -> 0
- net /ZB_TX: track 76.2 -> 68.1 mm
- net /RADAR_RX: track 47.4 -> 54.0 mm
- net /RF_CS: track 94.5 -> 88.7 mm
- net /+5V_C6: track 50.8 -> 55.8 mm
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Other:
- outline, holes or cut-outs redrawn
- board text added: "MC2-D ESP32"
- board text removed: "MC2-C ESP32"
