File: hardware/external-antenna/cad/mc2.kicad_sch (KiCad schematic)
At the start: 19 parts, among them J1 FUSED ISOLATED 5V INPUT, J2 D24V22F3 external assembled b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, J3 DFR0627 WK2132 ready module h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, J4 ZAC93 ready module harness, J5 CC1101 ready module harness, J6 LD2450 radar harness, J7 BME680 external pod harness, J8 XIAO BOOT unpopulated service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, J9 S3 BOOT unpopulated service p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, U1 ESP32-S3-DevKitC-1U-N8R8, U2 Unexpected Maker TinyC6-U-01, U3 Seeed XIAO MG24 pre-soldered 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, U4 WIZ850io finished module

Commit message: Migrate MC2-B to the lower-cost classic ESP32 host (#11)
Replace the MC2-A ESP32-S3-DevKitC-1U-N8R8 host with the
previous-generation ESP32-DevKitC-VIE / WROVER-IE to reduce host
purchase cost while retaining Ethernet, local OTBR, Zigbee, three active
BLE proxy connections, Z-Wave, RF RX/TX, LD2450 and BME680. The indexed
VIE offer was $9.48 versus the previously inspected $15.20 S3 promotion,
before delivery/tax; this is not a whole-device cost or power claim.

The new **MC2-B** carrier has the exact 38-pin host footprint, a checked
21-signal map and GPIO12/GPIO2 boot pull-downs. Keep the 100×100 mm
outline and supports, so the five existing enclosure meshes remain
unchanged. Update the schematic, routed PCB, connector lookup, BOM,
assembly instructions and README appearance concepts together.

Firmware targets classic ESP32 ECOv3 at 160 MHz, quad PSRAM at 40 MHz
and node identity `mc2-classic-hub`. Check actual image target/revision,
disable the IDF console so UART0 can serve radar, and preserve UART1/2
for Zigbee/Thread. Extend the shared component guards without changing
the S3 defaults. Fix the authenticated updater's expected node name and
bind its C6 evidence to the current recipe.

Compatibility limits are explicit: **BLE 4.2**, no BLE 5 extended
advertising or Coded PHY; 8 MB physical PSRAM but at most 4 MB directly
mapped. This requires the new carrier and an initial USB-UART flash with
private configuration. S3 OTA images and MC2-A pinouts are incompatible.
No hardware was flashed or Home Assistant changed.

Validation:
- Full pinned ESPHome 2026.9.1 / ESP-IDF 5.5.5 host build:
1,708,944-byte application; 2,223,216 bytes spare in each OTA slot;
separate DRAM/IRAM evidence and image-header checks.
- 26 MC2 tests, 62 MC1 regressions, 77 shared RF/UART/migration tests,
13 MG24 recipe tests; C++ RMT lifecycle checked with ASan/UBSan.
- KiCad ERC, DRC, unconnected items and schematic parity: zero; clean
CAD reproduction passes; every pin-plan role checked agai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
Parts:
- added R4: 10k host GPIO12 SCK boot pull-down, MC2:R_Axial_DIN0207_L6.3mm_D2.5mm_P7.62mm_Horizontal, symbol MC2:Module_R4
- added R5: 10k host GPIO2 MOSI boot pull-down, MC2:R_Axial_DIN0207_L6.3mm_D2.5mm_P7.62mm_Horizontal, symbol MC2:Module_R5
- J9: value S3 BOOT unpopulated service pads -> HOST BOOT unpopulated service pads
- U1: value ESP32-S3-DevKitC-1U-N8R8 -> ESP32-DevKitC-VIE; footprint MC2:S3_DevKitC1U -> MC2:ESP32_DevKitC_VIE
Connections:
- net ETH_CS: now also U1.J3.10 (GPIO5); no longer U1.J1.20 (GPIO14)
- net ETH_INT: now also U1.J2.5 (GPIO34); no longer U1.J1.16 (GPIO10)
- net ETH_RESET: now also U1.J3.13 (GPIO4); no longer U1.J1.15 (GPIO9)
- net GND: now also U1.J2.14 (GND), U1.J3.7 (GND), R4.1, R5.1; no longer U1.J1.22 (GND), U1.J3.21 (GND), U1.J3.22 (GND)
- net I2C_SCL: now also U1.J3.3 (GPIO22); no longer U1.J3.5 (GPIO2)
- net I2C_SDA: now also U1.J3.6 (GPIO21); no longer U1.J3.4 (GPIO1)
- net RADAR_RX: now also U1.J3.2 (GPIO23); no longer U1.J1.12 (GPIO8)
- net RADAR_TX: now also U1.J3.9 (GPIO18); no longer U1.J3.8 (GPIO40)
- net RF_CS: now also U1.J2.15 (GPIO13); no longer U1.J1.6 (GPIO6)
- net RF_GDO0: now also U1.J2.9 (GPIO25); no longer U1.J1.4 (GPIO4)
- net RF_GDO2: now also U1.J2.6 (GPIO35); no longer U1.J1.5 (GPIO5)
- net SPI_MISO: now also U1.J3.8 (GPIO19); no longer U1.J1.18 (GPIO12)
- net SPI_MOSI: now also U1.J3.15 (GPIO2), R5.2; no longer U1.J1.17 (GPIO11)
- net SPI_SCK: now also U1.J2.13 (GPIO12), R4.2; no longer U1.J1.19 (GPIO13)
- net THREAD_BOOT: now also U1.J3.16 (GPIO15); no longer U1.J3.9 (GPIO39)
- net THREAD_EN: now also U1.J2.11 (GPIO27); no longer U1.J3.17 (GPIO47)
- net THREAD_RX: now also U1.J2.10 (GPIO26); no longer U1.J1.8 (GPIO15)
- net THREAD_TX: now also U1.J2.3 (GPIO36); no longer U1.J1.9 (GPIO16)
- net ZB_CTS: now also U1.J2.8 (GPIO33); no longer U1.J1.7 (GPIO7)
- net ZB_RTS: now also U1.J2.12 (GPIO14); no longer U1.J3.18 (GPIO21)
- net ZB_RX: now also U1.J2.7 (GPIO32); no longer U1.J1.10 (GPIO17)
- net ZB_TX: now also U1.J2.4 (GPIO39); no longer U1.J1.11 (GPIO18)
- net +5V_S3 renamed +5V_HOST
- net +5V_HOST: now also U1.J2.19 (5V); no longer U1.J1.21 (5V)
- net S3_BOOT_SERVICE renamed HOST_BOOT_SERVICE
- no-connect marks 39 -> 34
Other:
- title: MC2 External antennas - engineering prototype -> MC2-B ESP32 external antennas - engineering prototype

Commit message: Match the MC2-C prototype to available TinyC6 D hardware (#17)
The original TC6-U-01 is obsolete/restricted at the checked US supplier
and has not been purchased. MC2-C selects the available TinyC6[D]
TC6D-01 and ships one matching carrier, firmware and enclosure package
for a five-board prototype order.

- Transcribe and verify the new module against pinned manufacturer
schematic, pinout and STEP files; correct its longer body, unused GPIO10
pad label, USB shell and relocated U.FL endpoint. Keep all connected
pads and copper unchanged.
- Select the external antenna through FXL6408 before Thread starts, fail
closed on configuration errors, and reject old C6 images in the updater.
Preserve the classic ESP32 host and all existing services.
- Regenerate the FH1 assembly views and print archive. All 14 printable
STL geometries remain unchanged; the corrected Thread coax route fits
the selected 150 mm cable with the specified slack.
- Publish native Gerbers, separate PTH/NPTH drill files and a manifest
that rejects stale CAD, firmware recipes, mechanical inputs and
artifacts. Add the ordering guide, current part availability and
observed quantity/shipping comparison.

Validation: native KiCad 10.0.6 ERC/DRC/unconnected/parity all zero;
clean source reproduction and unchanged-connected-copper comparison
pass. Fresh ESP32 and C6 builds pass. Firmware suites: 193 tests;
full-hub mechanics: 30 tests; fabrication/harness/guide: 24 tests.
Offline source/link/secret checks pass. Physical fit, rail headroom,
radio coexistence and coverage remain prototype commissioning work. No
purchase, device flash or Home Assistant migration has been performed.
Parts:
- U2: value Unexpected Maker TinyC6-U-01 -> Unexpected Maker TinyC6[D] TC6D-01; footprint MC2:TinyC6_U -> MC2:TinyC6_D
Other:
- title: MC2-B ESP32 external antennas - engineering prototype -> MC2-C ESP32 external antennas - engineering prototype
Changed lines of the file:
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@@
-(kicad_sch (version 20250114) (generator "eeschema") (paper "A3") (title_block (title "MC2-B ESP32 external antennas - engineering prototype") (date "2026-10-18") (rev "MC2-B") (comment 1 "Direct-solder THT male pins; all parts front; no carrier SMT") (comment 2 "External isolated fused 5V; separate peripheral 3V3; module 3V3 outputs never joined"))
+(kicad_sch (version 20250114) (generator "eeschema") (paper "A3") (title_block (title "MC2-C ESP32 external antennas - engineering prototype") (date "2026-10-19") (rev "MC2-C") (comment 1 "Direct-solder THT male pins; all parts front; no carrier SMT") (comment 2 "External isolated fused 5V; separate peripheral 3V3; module 3V3 outputs never joined"))
 (wire (pts (xy 25.4 35.56) (xy 20.32 35.56)) (stroke (width 0) (type default)))
 (wire (pts (xy 25.4 38.1) (xy 20.32 38.1)) (stroke (width 0) (type default)))
@@
 (symbol (lib_id "MC2:Module_U2") (at 147.3200 30.4800 0) (unit 1) (in_bom yes) (on_board yes) (dnp no)
 (property "Reference" "U2" (at 147.32 24.130000000000003 0) (effects (font (size 1.27 1.27))))
-(property "Value" "Unexpected Maker TinyC6-U-01" (at 147.32 26.67 0) (effects (font (size 1 1))))
-(property "Footprint" "MC2:TinyC6_U" (at 147.32 30.48 0) (effects (font (size 1 1)) hide))
+(property "Value" "Unexpected Maker TinyC6[D] TC6D-01" (at 147.32 26.67 0) (effects (font (size 1 1))))
+(property "Footprint" "MC2:TinyC6_D" (at 147.32 30.48 0) (effects (font (size 1 1)) hide))
 (pin "1")
 (pin "2")

Commit message: Migrate MC2-D to factory-header XIAO ESP32C6
Parts:
- removed R3: 10k C6 download strap GPIO8, MC2:R_Axial_DIN0207_L6.3mm_D2.5mm_P7.62mm_Horizontal, symbol MC2:Module_R3
- added J10: C6 EN/BOOT underside recovery harness, MC2:PinHeader_1x02_P2.54mm_Vertical, symbol MC2:Module_J10
- J2: value D24V22F3 external assembled buck -> RECOM R-78K3.3-1.0 offboard 3V3 converter
- U2: value Unexpected Maker TinyC6[D] TC6D-01 -> Seeed XIAO ESP32C6 pre-soldered 102010636; footprint MC2:TinyC6_D -> MC2:XIAO_ESP32C6
Connections:
- net +5V_C6: now also U2.14 (5V); no longer U2.3 (5V)
- net GND: now also U2.13 (GND); no longer U2.14 (GND), U2.2 (GND)
- net THREAD_BOOT: now also J10.2 (THREAD_BOOT); no longer U2.11 (GPIO9)
- net THREAD_EN: now also J10.1 (THREAD_EN); no longer U2.15 (EN)
- net THREAD_RX: now also U2.8 (GPIO17); no longer U2.12 (GPIO17)
- net THREAD_TX: now also U2.7 (GPIO16); no longer U2.13 (GPIO16)
- net C6_LOCAL_3V3: no longer names the net of U2.4 (GPIO21)
- net C6_STRAP8: no longer names the net of U2.10 (GPIO20)
- no-connect marks 34 -> 30
Other:
- title: MC2-C ESP32 external antennas - engineering prototype -> MC2-D ESP32 external antennas - engineering prototype
Changed lines of the file:
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@@
-(kicad_sch (version 20250114) (generator "eeschema") (paper "A3") (title_block (title "MC2-C ESP32 external antennas - engineering prototype") (date "2026-10-19") (rev "MC2-C") (comment 1 "Direct-solder THT male pins; all parts front; no carrier SMT") (comment 2 "External isolated fused 5V; separate peripheral 3V3; module 3V3 outputs never joined"))
+(kicad_sch (version 20250114) (generator "eeschema") (paper "A3") (title_block (title "MC2-D ESP32 external antennas - engineering prototype") (date "2026-10-20") (rev "MC2-D") (comment 1 "Direct-solder THT male pins; all parts front; no carrier SMT") (comment 2 "External isolated fused 5V; separate peripheral 3V3; module 3V3 outputs never joined"))
 (wire (pts (xy 25.4 35.56) (xy 20.32 35.56)) (stroke (width 0) (type default)))
 (wire (pts (xy 25.4 38.1) (xy 20.32 38.1)) (stroke (width 0) (type default)))
@@
 (wire (pts (xy 66.04 66.04) (xy 71.12 66.04)) (stroke (width 0) (type default)))
 (wire (pts (xy 66.04 68.58) (xy 71.12 68.58)) (stroke (width 0) (type default)))
-(wire (pts (xy 127.0 33.02) (xy 121.92 33.02)) (stroke (width 0) (type default)))
-(wire (pts (xy 127.0 35.56) (xy 121.92 35.56)) (stroke (width 0) (type default)))
-(wire (pts (xy 127.0 38.1) (xy 121.92 38.1)) (stroke (width 0) (type default)))
-(wire (pts (xy 127.0 53.34) (xy 121.92 53.34)) (stroke (width 0) (type default)))
-(wire (pts (xy 127.0 55.88) (xy 121.92 55.88)) (stroke (width 0) (type default)))
-(wire (pts (xy 127.0 58.42) (xy 121.92 58.42)) (stroke (width 0) (type default)))
+(wire (pts (xy 127.0 45.72) (xy 121.92 45.72)) (stroke (width 0) (type default)))
 (wire (pts (xy 167.64 30.48) (xy 172.72 30.48)) (stroke (width 0) (type default)))
-(wire (pts (xy 167.64 33.02) (xy 172.72 33.02)) (stroke (width 0) (type default)))
-(wire (pts (xy 167.64 35.56) (xy 172.72 35.56)) (stroke (width 0) (type default)))
+(wire (pts (xy 167.64 43.18) (xy 172.72 43.18)) (stroke (width 0) (type default)))
+(wire (pts (xy 167.64 45.72) (xy 172.72 45.72)) (stroke (width 0) (type default)))
 (wire (pts (xy 228.6 30.48) (xy 223.52 30.48)) (stroke (width 0) (type default)))
 (wire (pts (xy 228.6 40.64) (xy 223.52 40.64)) (stroke (width 0) (type default)))
@@
 (wire (pts (xy 228.6 246.38) (xy 223.52 246.38)) (stroke (width 0) (type default)))
 (wire (pts (xy 228.6 248.92) (xy 223.52 248.92)) (stroke (width 0) (type default)))
-(wire (pts (xy 342.9 246.38) (xy 337.82 246.38)) (stroke (width 0) (type default)))
-(wire (pts (xy 358.14 246.38) (xy 363.22 246.38)) (stroke (width 0) (type default)))
+(wire (pts (xy 330.2 246.38) (xy 325.12 246.38)) (stroke (width 0) (type default)))
+(wire (pts (xy 330.2 248.92) (xy 325.12 248.92)) (stroke (width 0) (type default)))
 (wire (pts (xy 38.1 281.94) (xy 33.02 281.94)) (stroke (width 0) (type default)))
 (wire (pts (xy 53.34 281.94) (xy 58.42 281.94)) (stroke (width 0) (type default)))
@@
 (label "SPI_MOSI" (at 71.12 66.04 0) (effects (font (size 0.9 0.9)) (justify left bottom)))
 (label "THREAD_BOOT" (at 71.12 68.58 0) (effects (font (size 0.9 0.9)) (justify left bottom)))
-(label "GND" (at 121.92 33.02 180) (effects (font (size 0.9 0.9)) (justify left bottom)))
-(label "+5V_C6" (at 121.92 35.56 180) (effects (font (size 0.9 0.9)) (justify left bottom)))
-(label "C6_LOCAL_3V3" (at 121.92 38.1 180) (effects (font (size 0.9 0.9)) (justify left bottom)))
-(label "C6_STRAP8" (at 121.92 53.34 180) (effects (font (size 0.9 0.9)) (justify left bottom)))
-(label "THREAD_BOOT" (at 121.92 55.88 180) (effects (font (size 0.9 0.9)) (justify left bottom)))
-(label "THREAD_RX" (at 121.92 58.42 180) (effects (font (size 0.9 0.9)) (justify left bottom)))
-(label "THREAD_TX" (at 172.72 30.48 0) (effects (font (size 0.9 0.9)) (justify left bottom)))
-(label "GND" (at 172.72 33.02 0) (effects (font (size 0.9 0.9)) (justify left bottom)))
-(label "THREAD_EN" (at 172.72 35.56 0) (effects (font (size 0.9 0.9)) (justify left bottom)))
+(label "THREAD_TX" (at 121.92 45.72 180) (effects (font (size 0.9 0.9)) (justify left bottom)))
+(label "THREAD_RX" (at 172.72 30.48 0) (effects (font (size 0.9 0.9)) (justify left bottom)))
+(label "GND" (at 172.72 43.18 0) (effects (font (size 0.9 0.9)) (justify left bottom)))
+(label "+5V_C6" (at 172.72 45.72 0) (effects (font (size 0.9 0.9)) (justify left bottom)))
 (label "ZB_BOOT_SERVICE" (at 223.52 30.48 180) (effects (font (size 0.9 0.9)) (justify left bottom)))
 (label "ZB_CTS" (at 223.52 40.64 180) (effects (font (size 0.9 0.9)) (justify left bottom)))
@@
 (label "HOST_BOOT_SERVICE" (at 223.52 246.38 180) (effects (font (size 0.9 0.9)) (justify left bottom)))
 (label "GND" (at 223.52 248.92 180) (effects (font (size 0.9 0.9)) (justify left bottom)))
-(label "C6_LOCAL_3V3" (at 337.82 246.38 180) (effects (font (size 0.9 0.9)) (justify left bottom)))
-(label "C6_STRAP8" (at 363.22 246.38 0) (effects (font (size 0.9 0.9)) (justify left bottom)))
+(label "THREAD_EN" (at 325.12 246.38 180) (effects (font (size 0.9 0.9)) (justify left bottom)))
+(label "THREAD_BOOT" (at 325.12 248.92 180) (effects (font (size 0.9 0.9)) (justify left bottom)))
 (label "GND" (at 33.02 281.94 180) (effects (font (size 0.9 0.9)) (justify left bottom)))
 (label "SPI_SCK" (at 58.42 281.94 0) (effects (font (size 0.9 0.9)) (justify left bottom)))
@@
 (no_connect (at 66.04 76.2))
 (no_connect (at 127.0 30.48))
+(no_connect (at 127.0 33.02))
+(no_connect (at 127.0 35.56))
+(no_connect (at 127.0 38.1))
 (no_connect (at 127.0 40.64))
 (no_connect (at 127.0 43.18))
-(no_connect (at 127.0 45.72))
-(no_connect (at 127.0 48.26))
-(no_connect (at 127.0 50.8))
+(no_connect (at 167.64 33.02))
+(no_connect (at 167.64 35.56))
 (no_connect (at 167.64 38.1))
 (no_connect (at 167.64 40.64))
-(no_connect (at 167.64 43.18))
-(no_connect (at 167.64 45.72))
-(no_connect (at 167.64 48.26))
-(no_connect (at 167.64 50.8))
-(no_connect (at 167.64 53.34))
-(no_connect (at 167.64 55.88))
 (no_connect (at 228.6 33.02))
 (no_connect (at 228.6 35.56))
@@
 (symbol (lib_id "MC2:Module_U2") (at 147.3200 30.4800 0) (unit 1) (in_bom yes) (on_board yes) (dnp no)
 (property "Reference" "U2" (at 147.32 24.130000000000003 0) (effects (font (size 1.27 1.27))))
-(property "Value" "Unexpected Maker TinyC6[D] TC6D-01" (at 147.32 26.67 0) (effects (font (size 1 1))))
-(property "Footprint" "MC2:TinyC6_D" (at 147.32 30.48 0) (effects (font (size 1 1)) hide))
+(property "Value" "Seeed XIAO ESP32C6 pre-soldered 102010636" (at 147.32 26.67 0) (effects (font (size 1 1))))
+(property "Footprint" "MC2:XIAO_ESP32C6" (at 147.32 30.48 0) (effects (font (size 1 1)) hide))
 (pin "1")
 (pin "2")
@@
 (pin "13")
 (pin "14")
-(pin "15")
-(pin "16")
-(pin "17")
-(pin "18")
-(pin "19")
-(pin "20")
-(pin "21")
-(pin "22")
-(pin "23")
 (instances (project "mc2" (path "/24581fcf-1632-59ed-8931-7790c5d2febc" (reference "U2") (unit 1)))))
 (symbol (lib_id "MC2:Module_U3") (at 248.9200 30.4800 0) (unit 1) (in_bom yes) (on_board yes) (dnp no)
@@
 (symbol (lib_id "MC2:Module_J2") (at 147.3200 111.7600 0) (unit 1) (in_bom yes) (on_board yes) (dnp no)
 (property "Reference" "J2" (at 147.32 105.41000000000001 0) (effects (font (size 1.27 1.27))))
-(property "Value" "D24V22F3 external assembled buck" (at 147.32 107.95 0) (effects (font (size 1 1))))
+(property "Value" "RECOM R-78K3.3-1.0 offboard 3V3 converter" (at 147.32 107.95 0) (effects (font (size 1 1))))
 (property "Footprint" "MC2:PinHeader_1x04_P2.54mm_Vertical" (at 147.32 111.76 0) (effects (font (size 1 1)) hide))
 (pin "1")
@@
 (pin "2")
 (instances (project "mc2" (path "/24581fcf-1632-59ed-8931-7790c5d2febc" (reference "J9") (unit 1)))))
-(symbol (lib_id "MC2:Module_R3") (at 350.5200 246.3800 0) (unit 1) (in_bom yes) (on_board yes) (dnp no)
-(property "Reference" "R3" (at 350.52 240.03 0) (effects (font (size 1.27 1.27))))
-(property "Value" "10k C6 download strap GPIO8" (at 350.52 242.57 0) (effects (font (size 1 1))))
-(property "Footprint" "MC2:R_Axial_DIN0207_L6.3mm_D2.5mm_P7.62mm_Horizontal" (at 350.52 246.38 0) (effects (font (size 1 1)) hide))
-(pin "1")
-(pin "2")
-(instances (project "mc2" (path "/24581fcf-1632-59ed-8931-7790c5d2febc" (reference "R3") (unit 1)))))
+(symbol (lib_id "MC2:Module_J10") (at 350.5200 246.3800 0) (unit 1) (in_bom yes) (on_board yes) (dnp no)
+(property "Reference" "J10" (at 350.52 240.03 0) (effects (font (size 1.27 1.27))))
+(property "Value" "C6 EN/BOOT underside recovery harness" (at 350.52 242.57 0) (effects (font (size 1 1))))
+(property "Footprint" "MC2:PinHeader_1x02_P2.54mm_Vertical" (at 350.52 246.38 0) (effects (font (size 1 1)) hide))
+(pin "1")
+(pin "2")
+(instances (project "mc2" (path "/24581fcf-1632-59ed-8931-7790c5d2febc" (reference "J10") (unit 1)))))
 (symbol (lib_id "MC2:Module_R4") (at 45.7200 281.9400 0) (unit 1) (in_bom yes) (on_board yes) (dnp no)
 (property "Reference" "R4" (at 45.72 275.59 0) (effects (font (size 1.27 1.27))))

Commit message: Qualify MC2-D purchase fit and remove host feed voltage drop
Parts:
- D1: value 1N5819 USB supply isolation -> 22AWG WIRE LINK - NO DIODE; footprint MC2:D_DO-41_SOD81_P7.62mm_Horizontal -> MC2:Wire_Link_P7.62mm
Changed lines of the file:
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@@
 (symbol (lib_id "MC2:Module_D1") (at 45.7200 210.8200 0) (unit 1) (in_bom yes) (on_board yes) (dnp no)
 (property "Reference" "D1" (at 45.72 204.47 0) (effects (font (size 1.27 1.27))))
-(property "Value" "1N5819 USB supply isolation" (at 45.72 207.01 0) (effects (font (size 1 1))))
-(property "Footprint" "MC2:D_DO-41_SOD81_P7.62mm_Horizontal" (at 45.72 210.82 0) (effects (font (size 1 1)) hide))
+(property "Value" "22AWG WIRE LINK - NO DIODE" (at 45.72 207.01 0) (effects (font (size 1 1))))
+(property "Footprint" "MC2:Wire_Link_P7.62mm" (at 45.72 210.82 0) (effects (font (size 1 1)) hide))
 (pin "1")
 (pin "2")
